Commit message: modif roue + test script

File: src/mapping/description/robot_core.xacro (robot description, xacro)
@@ -48,5 +48,5 @@
         <parent link="base_link"/>
         <child link="gh_wheel"/>
-        <origin xyz="0.1 0.1 0" rpy="-${pi/2} 0 0" />
+        <origin xyz="0.1 0.17 0" rpy="-${pi/2} 0 0" />
         <axis xyz="0 0 1"/>
     </joint>
@@ -54,9 +54,9 @@
         <visual>
             <geometry>
-                <cylinder radius="0.055" length="0.04"/>
+                <cylinder radius="0.055" length="0.07"/>
             </geometry>
             <material name="blue"/>
         </visual>
-        <xacro:inertial_cylinder mass="0.1" length="0.04" radius="0.055">
+        <xacro:inertial_cylinder mass="0.1" length="0.07" radius="0.055">
             <origin xyz="0 0 0" rpy="0 0 0"/>
         </xacro:inertial_cylinder>
@@ -66,5 +66,5 @@
         <parent link="base_link"/>
         <child link="gb_wheel"/>
-        <origin xyz="-0.1 0.1 0" rpy="-${pi/2} 0 0" />
+        <origin xyz="-0.1 0.17 0" rpy="-${pi/2} 0 0" />
         <axis xyz="0 0 1"/>
     </joint>
@@ -72,9 +72,9 @@
         <visual>
             <geometry>
-                <cylinder radius="0.055" length="0.04"/>
+                <cylinder radius="0.055" length="0.07"/>
             </geometry>
             <material name="blue"/>
         </visual>
-        <xacro:inertial_cylinder mass="0.1" length="0.04" radius="0.055">
+        <xacro:inertial_cylinder mass="0.1" length="0.07" radius="0.055">
             <origin xyz="0 0 0" rpy="0 0 0"/>
         </xacro:inertial_cylinder>
@@ -84,5 +84,5 @@
         <parent link="base_link"/>
         <child link="dh_wheel"/>
-        <origin xyz="0.1 -0.1 0" rpy="-${pi/2} 0 0" />
+        <origin xyz="0.1 -0.17 0" rpy="-${pi/2} 0 0" />
         <axis xyz="0 0 1"/>
     </joint>
@@ -90,9 +90,9 @@
         <visual>
             <geometry>
-                <cylinder radius="0.055" length="0.04"/>
+                <cylinder radius="0.055" length="0.07"/>
             </geometry>
             <material name="blue"/>
         </visual>
-        <xacro:inertial_cylinder mass="0.1" length="0.04" radius="0.055">
+        <xacro:inertial_cylinder mass="0.1" length="0.07" radius="0.055">
             <origin xyz="0 0 0" rpy="0 0 0"/>
         </xacro:inertial_cylinder>
@@ -102,5 +102,5 @@
         <parent link="base_link"/>
         <child link="db_wheel"/>
-        <origin xyz="-0.1 -0.1 0" rpy="-${pi/2} 0 0" />
+        <origin xyz="-0.1 -0.17 0" rpy="-${pi/2} 0 0" />
         <axis xyz="0 0 1"/>
     </joint>
@@ -108,9 +108,9 @@
         <visual>
             <geometry>
-                <cylinder radius="0.055" length="0.04"/>
+                <cylinder radius="0.055" length="0.07"/>
             </geometry>
             <material name="blue"/>
         </visual>
-        <xacro:inertial_cylinder mass="0.1" length="0.04" radius="0.055">
+        <xacro:inertial_cylinder mass="0.1" length="0.07" radius="0.055">
             <origin xyz="0 0 0" rpy="0 0 0"/>
         </xacro:inertial_cylinder>
