Commit message: re

File: install/mapping_pfr3/share/mapping_pfr3/description/robot_core.xacro (robot description, xacro)
@@ -45,8 +45,8 @@
     </link>
      <!-- ROUE Gauche Haut GH -->
-     <joint name="gh_wheel_joint" type="continuous">
+     <joint name="gh_wheel_joint" type="fixed">
         <parent link="base_link"/>
         <child link="gh_wheel"/>
-        <origin xyz="0.1 0.1 0" rpy="-${pi/2} 0 0" />
+        <origin xyz="0.1 0.17 0" rpy="-${pi/2} 0 0" />
         <axis xyz="0 0 1"/>
     </joint>
@@ -54,17 +54,17 @@
         <visual>
             <geometry>
-                <cylinder radius="0.055" length="0.04"/>
+                <cylinder radius="0.055" length="0.07"/>
             </geometry>
             <material name="blue"/>
         </visual>
-        <xacro:inertial_cylinder mass="0.1" length="0.04" radius="0.055">
+        <xacro:inertial_cylinder mass="0.1" length="0.07" radius="0.055">
             <origin xyz="0 0 0" rpy="0 0 0"/>
         </xacro:inertial_cylinder>
     </link>
      <!-- ROUE GB -->
-     <joint name="gb_wheel_joint" type="continuous">
+     <joint name="gb_wheel_joint" type="fixed">
         <parent link="base_link"/>
         <child link="gb_wheel"/>
-        <origin xyz="-0.1 0.1 0" rpy="-${pi/2} 0 0" />
+        <origin xyz="-0.1 0.17 0" rpy="-${pi/2} 0 0" />
         <axis xyz="0 0 1"/>
     </joint>
@@ -72,17 +72,17 @@
         <visual>
             <geometry>
-                <cylinder radius="0.055" length="0.04"/>
+                <cylinder radius="0.055" length="0.07"/>
             </geometry>
             <material name="blue"/>
         </visual>
-        <xacro:inertial_cylinder mass="0.1" length="0.04" radius="0.055">
+        <xacro:inertial_cylinder mass="0.1" length="0.07" radius="0.055">
             <origin xyz="0 0 0" rpy="0 0 0"/>
         </xacro:inertial_cylinder>
     </link>
     <!-- ROUE DH -->
-    <joint name="dh_wheel_joint" type="continuous">
+    <joint name="dh_wheel_joint" type="fixed">
         <parent link="base_link"/>
         <child link="dh_wheel"/>
-        <origin xyz="0.1 -0.1 0" rpy="-${pi/2} 0 0" />
+        <origin xyz="0.1 -0.17 0" rpy="-${pi/2} 0 0" />
         <axis xyz="0 0 1"/>
     </joint>
@@ -90,17 +90,17 @@
         <visual>
             <geometry>
-                <cylinder radius="0.055" length="0.04"/>
+                <cylinder radius="0.055" length="0.07"/>
             </geometry>
             <material name="blue"/>
         </visual>
-        <xacro:inertial_cylinder mass="0.1" length="0.04" radius="0.055">
+        <xacro:inertial_cylinder mass="0.1" length="0.07" radius="0.055">
             <origin xyz="0 0 0" rpy="0 0 0"/>
         </xacro:inertial_cylinder>
     </link>
     <!-- ROUE DB -->
-    <joint name="db_wheel_joint" type="continuous">
+    <joint name="db_wheel_joint" type="fixed">
         <parent link="base_link"/>
         <child link="db_wheel"/>
-        <origin xyz="-0.1 -0.1 0" rpy="-${pi/2} 0 0" />
+        <origin xyz="-0.1 -0.17 0" rpy="-${pi/2} 0 0" />
         <axis xyz="0 0 1"/>
     </joint>
@@ -108,9 +108,9 @@
         <visual>
             <geometry>
-                <cylinder radius="0.055" length="0.04"/>
+                <cylinder radius="0.055" length="0.07"/>
             </geometry>
             <material name="blue"/>
         </visual>
-        <xacro:inertial_cylinder mass="0.1" length="0.04" radius="0.055">
+        <xacro:inertial_cylinder mass="0.1" length="0.07" radius="0.055">
             <origin xyz="0 0 0" rpy="0 0 0"/>
         </xacro:inertial_cylinder>
