Commit message: mapping marche

File: install/mapping_pfr3/share/mapping_pfr3/description/lidar.xacro (robot description, xacro)
@@ -4,5 +4,5 @@
         <parent link="chassis"/>
         <child link="laser_frame"/>
-        <origin xyz="0.125 0 0.06" rpy="0 0 0"/>
+        <origin xyz="0.125 0 0.05" rpy="0 0 0"/>
     </joint>
     <link name="laser_frame">

File: install/mapping_pfr3/share/mapping_pfr3/description/robot_core.xacro (robot description, xacro)
@@ -48,5 +48,5 @@
         <parent link="base_link"/>
         <child link="gh_wheel"/>
-        <origin xyz="0.1 0.17 0" rpy="-${pi/2} 0 0" />
+        <origin xyz="0.1 0.135 0" rpy="-${pi/2} 0 0" />
         <axis xyz="0 0 1"/>
     </joint>
@@ -54,5 +54,5 @@
         <visual>
             <geometry>
-                <cylinder radius="0.055" length="0.07"/>
+                <cylinder radius="0.0575" length="0.07"/>
             </geometry>
             <material name="blue"/>
@@ -66,5 +66,5 @@
         <parent link="base_link"/>
         <child link="gb_wheel"/>
-        <origin xyz="-0.1 0.17 0" rpy="-${pi/2} 0 0" />
+        <origin xyz="-0.1 0.135 0" rpy="-${pi/2} 0 0" />
         <axis xyz="0 0 1"/>
     </joint>
@@ -72,5 +72,5 @@
         <visual>
             <geometry>
-                <cylinder radius="0.055" length="0.07"/>
+                <cylinder radius="0.0575" length="0.07"/>
             </geometry>
             <material name="blue"/>
@@ -84,5 +84,5 @@
         <parent link="base_link"/>
         <child link="dh_wheel"/>
-        <origin xyz="0.1 -0.17 0" rpy="-${pi/2} 0 0" />
+        <origin xyz="0.1 -0.135 0" rpy="-${pi/2} 0 0" />
         <axis xyz="0 0 1"/>
     </joint>
@@ -90,5 +90,5 @@
         <visual>
             <geometry>
-                <cylinder radius="0.055" length="0.07"/>
+                <cylinder radius="0.0575" length="0.07"/>
             </geometry>
             <material name="blue"/>
@@ -102,5 +102,5 @@
         <parent link="base_link"/>
         <child link="db_wheel"/>
-        <origin xyz="-0.1 -0.17 0" rpy="-${pi/2} 0 0" />
+        <origin xyz="-0.1 -0.135 0" rpy="-${pi/2} 0 0" />
         <axis xyz="0 0 1"/>
     </joint>
@@ -108,5 +108,5 @@
         <visual>
             <geometry>
-                <cylinder radius="0.055" length="0.07"/>
+                <cylinder radius="0.0575" length="0.07"/>
             </geometry>
             <material name="blue"/>
